File: MD201x.sch (EAGLE design)
At the start: 103 parts, among them IC1 78L05F, IC2 LM321MF, J1 8P8C-LED, J10 1744446-4, J2 1744446-4, J3 XH-4-SIDE, J4 MA04-2, J5 MA05-2, J6 MA02-2, Q1 N-MOSFET-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

Commit message: 横向き
Parts:
- removed C35: 22u, rcl:CPOL-EUE2.5-5
- removed U11, U12, U13, U14, U15: 74AHC1G08DCK, 74xx-little-us:74AHC1G08DCK
- added D2, D3, D5, D6: (no value), diode:DIODE-SOD523
- added Q5: BSS123, transistor-small-signal:BSS123
- added R19: 0.5m, r_shunt:CSS2H-2512
- C33: device rcl:C-EUC0805 -> rcl:C-EUC0603
- C36: device rcl:C-EUC0603 -> rcl:C-EUC1210
- U$1: value XT60PW -> XT60PW-M; device lib_ysk:XT60PW -> lib_ysk:XT60PW-M
- U$2: value XT60PW -> XT60PW-F; device lib_ysk:XT60PW -> lib_ysk:XT60PW-F
Connections:
- net N$23 renamed CANTX_ISO
- net N$27 renamed CANRX_ISO
- net VCS_N renamed VCS_B_N
- net VCS_P renamed VCS_B_P
- removed net 24V_ISO: C35.+, C36.1, IC1.VI, J1.4, J1.5, R20.1
- removed net VCS: C11.2, C12.2, C5.2, C6.2, Q2.SOURCE, Q4.SOURCE, R7.1, R8.1, R9.2
- new net A_LS: Q2.SOURCE, R19.2, R7.1
- new net B_LS: C6.2, Q4.SOURCE, R8.1, R9.2
- new net DC_ISO: C36.1, IC1.VI, J1.4, J1.5, R20.1
- new net ISENSE_B: C16.2, R123.1
- new net N$13: J6.1
- net !EMS: no longer U12A.I0, U13A.I0, U14A.I0, U15A.I0
- net +3V3: no longer U12P.VCC, U13P.VCC, U14P.VCC, U15P.VCC
- net 5V_ISO: now also R17.2; no longer U11P.VCC
- net CANH: no longer J6.1
- net CANL: no longer R12.1
- net GNDA: now also C11.2, C12.2, C5.2, R19.1; no longer U12P.GND, U13P.GND, U14P.GND, U15P.GND
- net GNDIO: now also Q5.S; no longer C35.-, R17.1, U11P.GND
- net IN_HI_A: no longer U13A.O
- net IN_HI_A_PRE: no longer U13A.I1
- net IN_HI_B: no longer U14A.O
- net IN_HI_B_PRE: no longer U14A.I1
- net IN_LO_A: no longer U12A.O
- net IN_LO_A_PRE: no longer U12A.I1
- net IN_LO_B: no longer U15A.O
- net IN_LO_B_PRE: no longer U15A.I1
- net ISENSE: no longer C16.2, R123.1
- net N$1: now also D6.C
- net N$11: now also D5.C
- net N$12: now also D2.A
- net N$16: now also R17.1; no longer U11A.O
- net N$17: now also Q5.D; no longer R17.2
- net N$2: now also D2.C
- net N$4: now also D6.A
- net N$5: now also D3.C
- net N$61: now also D5.A
- net N$64: now also D3.A
- net N$8: now also Q5.G; no longer U11A.I0, U11A.I1
Other:
- note added: "TODO: BOOT0をジャンパで切り替えられるようにする"
- note added: "TODO: PWM信号を直列終端する"
- note added: "TODO: エンコーダ入力を5Vトレラントにする"
- note added: "TODO: デバッガ用コネクタを最適化する"
- moved on the sheet: C10, C11, C12, C14, C15, C16, C17, C5, C6, C8, C9, D4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

Commit message: staging everything i have right now
Parts:
- removed U7: NCS199, on-semi:NCS199
- added C31: (no value), rcl:C-EUC0603
- added CN2: (no value), jst-xa:S3B-XASK-1
- added R22, R23: 10, rcl:R-EU_R0603
- added U$3: INA186DCK, lib_ysk:INA186DCK
- U5: value NCP5106D -> NCP5106MN; device on-semi:NCP5106D -> on-semi:NCP5106MN
- U6: value NCP5106D -> NCP5106; device on-semi:NCP5106D -> on-semi:NCP5106
Connections:
- new net 0V: C11.2, C12.2, C5.2, R19.1, R9.1
- new net N$15: C31.2, R22.2, U$3.IN-
- new net N$22: C31.1, R23.2, U$3.IN+
- net 3V3A: now also U$3.VS; no longer U7.VS
- net GNDA: now also U$3.GND; no longer C11.2, C12.2, C5.2, R19.1, R9.1, U7.GND
- net N$6: no longer U7.OUT
- net REF: no longer U7.REF
- net VCS_B_N: now also R22.1; no longer U7.IN-
- net VCS_B_P: now also R23.1; no longer U7.IN+
Other:
- moved on the sheet: C14, C15, C16, R123, R15, R16, U5

Commit message: idk
Parts:
- removed J10, J2: 1744446-4, con-ep25:1744446-4
- removed J3: XH-4-SIDE, con-xh:XH-4-SIDE
Connections:
- new net CS_OUT_A: U$3.OUT
- new net CS_REF: U$3.REF
- net +5V: no longer J10P2.1, J3.2
- net ENC_A: no longer J10P3.1
- net ENC_B: no longer J10P4.1
- net GNDA: no longer J10P1.1, J3.1
- net IN_A: no longer J3.3
- net IN_B: no longer J3.4

Commit message: stage everything
Parts:
- removed D4: BAS16W, diode:DIODE-SOD323-R
- removed U6: NCP5106, on-semi:NCP5106
- added U$4: DGD05473FN, lib_ysk:DGD05473FN
Connections:
- net +15V: now also U$4.VCC; no longer D4.A, U6.VCC
- net B_OUT: now also U$4.VS; no longer U6.BRIDGE
- net GNDA: now also U$4.COM; no longer U6.GND
- net IN_HI_B: now also U$4.HIN; no longer U6.IN_HI
- net IN_LO_B: now also U$4.LIN; no longer U6.IN_LO
- net N$2: now also U$4.HO; no longer U6.DRV_HI
- net N$5: now also U$4.LO; no longer U6.DRV_LO
- net N$67: now also U$4.VB; no longer D4.C, U6.VBOOT
Other:
- moved on the sheet: C10
Changed lines of the file:
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@@
 <part name="Q3" library="nexperia" deviceset="N-MOSFET-*" device="" value="N-MOSFET-"/>
 <part name="Q4" library="nexperia" deviceset="N-MOSFET-*" device="" value="N-MOSFET-"/>
-<part name="D4" library="diode" library_urn="urn:adsk.eagle:library:210" deviceset="DIODE-" device="SOD323-R" package3d_urn="urn:adsk.eagle:package:43437/1" value="BAS16W"/>
 <part name="C10" library="rcl" deviceset="C-EU" device="C0603" value="100n/25V"/>
 <part name="C11" library="rcl" deviceset="C-EU" device="C1210" value="10u"/>
@@
 <part name="U10" library="torex" deviceset="XC6206" device="" package3d_urn="urn:adsk.eagle:package:6993131/1"/>
 <part name="U5" library="on-semi" deviceset="NCP5106" device="MN" package3d_urn="urn:adsk.eagle:package:12418013/1" value="NCP5106MN"/>
-<part name="U6" library="on-semi" deviceset="NCP5106" device="" package3d_urn="urn:adsk.eagle:package:15356/1" value="NCP5106"/>
 <part name="R9" library="r_shunt" deviceset="CSS2H-2512" device="" value="0.5m"/>
 <part name="P+6" library="supply1" library_urn="urn:adsk.eagle:library:371" deviceset="VCC" device=""/>
@@
 <part name="R23" library="rcl" deviceset="R-EU_" device="R0603" value="10"/>
 <part name="C31" library="rcl" library_urn="urn:adsk.eagle:library:334" deviceset="C-EU" device="C0603" package3d_urn="urn:adsk.eagle:package:23616/2"/>
+<part name="U$4" library="lib_ysk" deviceset="DGD05473" device="FN" package3d_urn="urn:adsk.eagle:package:12826382/1"/>
 </parts>
 <sheets>
@@
 <attribute name="VALUE" x="82.55" y="20.32" size="1.778" layer="96"/>
 </instance>
-<instance part="D4" gate="G$1" x="12.7" y="48.26" smashed="yes">
-<attribute name="NAME" x="15.24" y="48.7426" size="1.778" layer="95"/>
-<attribute name="VALUE" x="15.24" y="45.9486" size="1.778" layer="96"/>
-</instance>
-<instance part="C10" gate="G$1" x="40.64" y="40.64" smashed="yes">
-<attribute name="NAME" x="42.164" y="41.021" size="1.778" layer="95"/>
-<attribute name="VALUE" x="42.164" y="35.941" size="1.778" layer="96"/>
+<instance part="C10" gate="G$1" x="35.56" y="38.1" smashed="yes" rot="R90">
+<attribute name="NAME" x="35.179" y="39.624" size="1.778" layer="95" rot="R90"/>
+<attribute name="VALUE" x="40.259" y="39.624" size="1.778" layer="96" rot="R90"/>
 </instance>
 <instance part="P+1" gate="VCC" x="78.74" y="144.78" smashed="yes">
@@
 <attribute name="VALUE" x="5.08" y="109.22" size="1.778" layer="96"/>
 </instance>
-<instance part="U6" gate="G$1" x="12.7" y="30.48" smashed="yes">
-<attribute name="NAME" x="5.08" y="41.91" size="1.778" layer="95"/>
-<attribute name="VALUE" x="5.08" y="17.78" size="1.778" layer="96"/>
-</instance>
 <instance part="R9" gate="G$1" x="78.74" y="-2.54" smashed="yes" rot="MR90">
 <attribute name="NAME" x="80.2386" y="-6.35" size="1.778" layer="95" rot="MR90"/>
@@
 <attribute name="VALUE" x="-43.18" y="106.68" size="1.778" layer="96" rot="R90"/>
 </instance>
-<instance part="GND7" gate="1" x="-5.08" y="17.78" smashed="yes">
-<attribute name="VALUE" x="-7.62" y="15.24" size="1.778" layer="96" rot="R90"/>
+<instance part="GND7" gate="1" x="-5.08" y="10.16" smashed="yes">
+<attribute name="VALUE" x="-7.62" y="7.62" size="1.778" layer="96" rot="R90"/>
 </instance>
 <instance part="GND8" gate="1" x="-35.56" y="17.78" smashed="yes">
@@
 <attribute name="VALUE" x="191.516" y="-51.181" size="1.778" layer="96" rot="R180"/>
 </instance>
+<instance part="U$4" gate="G$1" x="12.7" y="27.94" smashed="yes"/>
 </instances>
 <busses>
@@
 </segment>
 <segment>
-<pinref part="D4" gate="G$1" pin="A"/>
 <pinref part="SUPPLY20" gate="1" pin="+15V"/>
-<wire x1="10.16" y1="48.26" x2="-5.08" y2="48.26" width="0.1524" layer="91"/>
-<pinref part="U6" gate="G$1" pin="VCC"/>
 <wire x1="-5.08" y1="48.26" x2="-10.16" y2="48.26" width="0.1524" layer="91"/>
 <wire x1="0" y1="38.1" x2="-5.08" y2="38.1" width="0.1524" layer="91"/>
 <wire x1="-5.08" y1="38.1" x2="-5.08" y2="48.26" width="0.1524" layer="91"/>
-<junction x="-5.08" y="48.26"/>
 <pinref part="C8" gate="G$1" pin="1"/>
 <wire x1="-35.56" y1="38.1" x2="-5.08" y2="38.1" width="0.1524" layer="91"/>
 <wire x1="-35.56" y1="33.02" x2="-35.56" y2="38.1" width="0.1524" layer="91"/>
 <junction x="-5.08" y="38.1"/>
+<pinref part="U$4" gate="G$1" pin="VCC"/>
 </segment>
 <segment>
@@
 </segment>
 <segment>
-<wire x1="-5.08" y1="20.32" x2="-5.08" y2="22.86" width="0.1524" layer="91"/>
-<wire x1="-5.08" y1="22.86" x2="0" y2="22.86" width="0.1524" layer="91"/>
-<pinref part="U6" gate="G$1" pin="GND"/>
+<wire x1="-5.08" y1="12.7" x2="-5.08" y2="17.78" width="0.1524" layer="91"/>
+<wire x1="-5.08" y1="17.78" x2="0" y2="17.78" width="0.1524" layer="91"/>
 <pinref part="GND7" gate="1" pin="GNDA"/>
+<pinref part="U$4" gate="G$1" pin="COM"/>
 </segment>
 <segment>
@@
 <net name="B_OUT" class="0">
 <segment>
-<wire x1="40.64" y1="27.94" x2="25.4" y2="27.94" width="0.1524" layer="91"/>
-<wire x1="40.64" y1="35.56" x2="40.64" y2="27.94" width="0.1524" layer="91"/>
+<wire x1="48.26" y1="27.94" x2="25.4" y2="27.94" width="0.1524" layer="91"/>
+<wire x1="40.64" y1="38.1" x2="48.26" y2="38.1" width="0.1524" layer="91"/>
+<wire x1="48.26" y1="38.1" x2="48.26" y2="27.94" width="0.1524" layer="91"/>
 <pinref part="C10" gate="G$1" pin="2"/>
 <wire x1="78.74" y1="35.56" x2="78.74" y2="33.02" width="0.1524" layer="91"/>
@@
 <wire x1="78.74" y1="33.02" x2="78.74" y2="27.94" width="0.1524" layer="91"/>
 <wire x1="78.74" y1="27.94" x2="78.74" y2="25.4" width="0.1524" layer="91"/>
-<wire x1="40.64" y1="27.94" x2="78.74" y2="27.94" width="0.1524" layer="91"/>
-<junction x="40.64" y="27.94"/>
+<wire x1="48.26" y1="27.94" x2="78.74" y2="27.94" width="0.1524" layer="91"/>
+<junction x="48.26" y="27.94"/>
 <junction x="78.74" y="27.94"/>
 <label x="68.58" y="27.94" size="1.778" layer="95"/>
-<pinref part="U6" gate="G$1" pin="BRIDGE"/>
 <pinref part="R6" gate="G$1" pin="1"/>
 <wire x1="68.58" y1="33.02" x2="78.74" y2="33.02" width="0.1524" layer="91"/>
 <junction x="78.74" y="33.02"/>
+<pinref part="U$4" gate="G$1" pin="VS"/>
 </segment>
 <segment>
@@
 <net name="N$67" class="0">
 <segment>
-<wire x1="30.48" y1="48.26" x2="15.24" y2="48.26" width="0.1524" layer="91"/>
-<wire x1="40.64" y1="43.18" x2="40.64" y2="48.26" width="0.1524" layer="91"/>
-<wire x1="40.64" y1="48.26" x2="30.48" y2="48.26" width="0.1524" layer="91"/>
-<junction x="30.48" y="48.26"/>
-<pinref part="D4" gate="G$1" pin="C"/>
-<wire x1="30.48" y1="48.26" x2="30.48" y2="38.1" width="0.1524" layer="91"/>
-<wire x1="30.48" y1="38.1" x2="25.4" y2="38.1" width="0.1524" layer="91"/>
+<wire x1="33.02" y1="38.1" x2="25.4" y2="38.1" width="0.1524" layer="91"/>
 <pinref part="C10" gate="G$1" pin="1"/>
-<pinref part="U6" gate="G$1" pin="VBOOT"/>
+<pinref part="U$4" gate="G$1" pin="VB"/>
 </segment>
 </net>
@@
 <wire x1="58.42" y1="12.7" x2="55.88" y2="12.7" width="0.1524" layer="91"/>
 <wire x1="55.88" y1="12.7" x2="55.88" y2="17.78" width="0.1524" layer="91"/>
-<pinref part="U6" gate="G$1" pin="DRV_LO"/>
 <wire x1="25.4" y1="22.86" x2="55.88" y2="22.86" width="0.1524" layer="91"/>
 <junction x="55.88" y="22.86"/>
 <pinref part="D3" gate="G$1" pin="C"/>
+<pinref part="U$4" gate="G$1" pin="LO"/>
 </segment>
 </net>
@@
 <wire x1="58.42" y1="33.02" x2="55.88" y2="33.02" width="0.1524" layer="91"/>
 <junction x="55.88" y="33.02"/>
-<pinref part="U6" gate="G$1" pin="DRV_HI"/>
 <pinref part="D2" gate="G$1" pin="C"/>
+<pinref part="U$4" gate="G$1" pin="HO"/>
 </segment>
 </net>
@@
 <net name="IN_LO_B" class="0">
 <segment>
-<pinref part="U6" gate="G$1" pin="IN_LO"/>
 <wire x1="0" y1="27.94" x2="-17.78" y2="27.94" width="0.1524" layer="91"/>
 <label x="-20.32" y="27.94" size="1.778" layer="95"/>
+<pinref part="U$4" gate="G$1" pin="LIN"/>
 </segment>
 </net>
@@
 <wire x1="0" y1="33.02" x2="-17.78" y2="33.02" width="0.1524" layer="91"/>
 <label x="-20.32" y="33.02" size="1.778" layer="95"/>
-<pinref part="U6" gate="G$1" pin="IN_HI"/>
-</segment>
-</net>
+<pinref part="U$4" gate="G$1" pin="HIN"/>
+</segment>
+</net>
