File: MD201x.brd (EAGLE design)
At the start: 100 x 50 mm, 105 parts, among them IC1 78L05F, IC2 LM321MF, J1 8P8C-LED, J4 MA04-2, J5 MA05-2, J6 MA02-2, Q1 N-MOSFET-, Q2 N-MOSFET-, Q3 N-MOSFET-, Q4 N-MOSFET-, Q5 BSS123, U1 STM32F303C, U10 XC6206, U2 NCV7351D1E, U3 SI8621AB-B-IS, U4 TLP184, U5 NCP5106MN, U8 7815DT, U9 7805DT, X1 CSTCE8M00G55

Commit message: still in progress...
Parts:
- moved D2 72.9 mm to (87.3, -24.8), turned to 180 degrees
- moved U$3 71.5 mm to (80.0, -24.5), turned to 180 degrees
- moved R2 69.0 mm to (87.4, -22.8), turned to 180 degrees
- moved D3 66.6 mm to (77.8, -21.9), turned to 180 degrees
- moved R23 66.5 mm to (79.5, -22.0), turned to 180 degrees
- moved R8 65.3 mm to (75.1, -20.8), turned to 270 degrees
- moved R6 64.6 mm to (87.4, -20.6), turned to 0 degrees
- moved C31 64.4 mm to (82.1, -21.0), turned to 90 degrees
- moved U$4 64.3 mm to (83.4, -20.9), turned to 90 degrees
- moved R4 63.3 mm to (77.8, -20.2), turned to 180 degrees
- moved R22 62.3 mm to (79.5, -19.9), turned to 180 degrees
- moved C2 54.1 mm to (94.0, 15.4), turned to 0 degrees
- moved R9 52.1 mm to (79.8, -14.8), turned to 90 degrees
- moved C12 49.5 mm to (85.6, -13.2), turned to 270 degrees
- moved C6 46.9 mm to (83.0, -12.2), turned to 270 degrees
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Routing:
- net B_OUT: track 17.7 -> 0.00 mm
- net N$12: track 15.4 -> 0.00 mm
- net N$11: track 10.3 -> 0.00 mm
- net N$61: track 3.76 -> 0.00 mm
- net GNDA: vias 54 -> 41
- removed copper zone on layer 16, net A_OUT
- removed copper zone on layer 16, net B_OUT
